Commit message: update

File: urdf/model.xacro (robot description, xacro)
@@ -11,5 +11,5 @@
                <inertial>
                        <mass value="${mass}" />
-                       <inertia ixx="0.0045" ixy="0" ixz="0" iyy="0.005" iyz="0" izz="0.0045" />
+                       <inertia ixx="0.0045" ixy="0" ixz="0" iyy="0.0045" iyz="0" izz="0.0045" />
                </inertial>
     </xacro:macro>
@@ -46,5 +46,5 @@
         <inertial>
             <mass value="35" />
-            <inertia ixx="0.6125" ixy="0.00495" ixz="0.0031" iyy="0.6426" iyz="-0.0017" izz="0.494" />
+            <inertia ixx="0.45" ixy="0.000" ixz="0.000" iyy="0.55" iyz="0.000" izz="0.6125" />
         </inertial>
     </link>
@@ -201,5 +201,5 @@
             <odometryFrame>${ns}odom</odometryFrame>
             <torque>15</torque>
-            <topicName>${ns}cmd_vel</topicName>
+            <topicName>cmd_vel</topicName>
             <broadcastTF>1</broadcastTF>
         </plugin>
@@ -231,6 +231,6 @@
             </ray>
             <plugin name="gazebo_ros_head_hokuyo_controller" filename="libgazebo_ros_laser.so">
-                <topicName>${ns}scan</topicName>
-                <frameName>${ns}hokuyo_link</frameName>
+                <topicName>scan</topicName>
+                <frameName>hokuyo_link</frameName>
             </plugin>
         </sensor>

Commit message: deleted usless map and add check input coordinate feature

File: urdf/model.xacro (robot description, xacro)
@@ -32,5 +32,5 @@
             <geometry>
                     <box size="0.2 .3 .1"/>
-                </geometry>
+            </geometry>
             <origin rpy="0 0 1.571" xyz="0 0 0.05"/>
             <material name="white">
@@ -200,5 +200,5 @@
             <robotBaseFrame>${ns}base_footprint</robotBaseFrame>
             <odometryFrame>${ns}odom</odometryFrame>
-            <torque>15</torque>
+            <torque>20</torque>
             <topicName>cmd_vel</topicName>
             <broadcastTF>1</broadcastTF>

Commit message: add hokuyo mesh file so that it can run without other package

File: urdf/model.xacro (robot description, xacro)
@@ -119,5 +119,5 @@
             <origin xyz="0 0 0" rpy="0 0 0" />
             <geometry>
-                <mesh filename="package://robot1_description/meshes/hokuyo.dae" />
+                <mesh filename="package://multiple_rb_ctrl/urdf/hokuyo.dae" />
             </geometry>
         </visual>

Commit message: changed urdf to make model easier to control

File: urdf/model.xacro (robot description, xacro)
@@ -31,7 +31,7 @@
         <visual>
             <geometry>
-                    <box size="0.2 .3 .1"/>
-            </geometry>
-            <origin rpy="0 0 1.571" xyz="0 0 0.05"/>
+                    <box size="0.2 0.3 0.1"/>
+            </geometry>
+            <origin rpy="0 0 1.571" xyz="0 0 0.00"/>
             <material name="white">
                 <color rgba="1 1 1 1"/>
@@ -40,7 +40,7 @@
         <collision>
             <geometry>
-                    <box size="0.2 .3 0.1"/>
-            </geometry>
-            <origin rpy="0 0 1.571" xyz="0 0 0.05"/>
+                    <box size="0.2 0.3 0.1"/>
+            </geometry>
+            <origin rpy="0 0 1.571" xyz="0 0 0.00"/>
         </collision>
         <inertial>
@@ -83,10 +83,9 @@
         <xacro:default_inertial mass="4.3542"/>
     </link>
-    <link name="${ns}wheel_3">
-        <visual>
-                <geometry>
-                    <cylinder length="${length_wheel}" radius="${radius_wheel}"/>
-                </geometry>
-            <!-- <origin rpy="0 1.5 0" xyz="0.1 -0.1 0"/> -->
+    <link name="${ns}front_omni">
+        <visual>
+                <geometry>
+                    <sphere radius="0.0125"/>
+                </geometry>
             <origin rpy="0 0 0" xyz="0 0 0"/>
             <material name="black"/>
@@ -94,15 +93,24 @@
         <collision>
             <geometry>
-                    <cylinder length="${length_wheel}" radius="${radius_wheel}"/>
-            </geometry>
-        </collision>
-        <xacro:default_inertial mass="4.3542"/>
-    </link>
-    <link name="${ns}wheel_4">
-        <visual>
-                <geometry>
-                    <cylinder length="${length_wheel}" radius="${radius_wheel}"/>
-                </geometry>
-        <!--    <origin rpy="0 1.5 0" xyz="-0.1 -0.1 0"/> -->
+                   <sphere radius="0.0124"/>
+            </geometry>
+            <surface>
+              <friction>
+                <ode>
+                  <mu>0</mu>
+                  <mu2>0</mu2>
+                  <slip1>1.0</slip1>
+                  <slip2>1.0</slip2>
+                </ode>
+              </friction>
+            </surface>
+        </collision>
+        <xacro:default_inertial mass="1"/>
+    </link>
+    <link name="${ns}back_omni">
+        <visual>
+                <geometry>
+                    <sphere radius="0.0125"/>
+                </geometry>
             <origin rpy="0 0 0" xyz="0 0 0" />
             <material name="black"/>
@@ -110,8 +118,18 @@
         <collision>
             <geometry>
-                    <cylinder length="${length_wheel}" radius="${radius_wheel}"/>
-            </geometry>
-        </collision>
-        <xacro:default_inertial mass="4.3542"/>
+                   <sphere radius="0.0124"/>
+            </geometry>
+            <surface>
+              <friction>
+                <ode>
+                  <mu>0</mu>
+                  <mu2>0</mu2>
+                  <slip1>1.0</slip1>
+                  <slip2>1.0</slip2>
+                </ode>
+              </friction>
+            </surface>
+        </collision>
+        <xacro:default_inertial mass="1"/>
     </link>
     <link name="${ns}hokuyo_link">
@@ -135,28 +153,24 @@
     </link>
     <joint name="${ns}base_to_wheel1" type="continuous">
-    <parent link="${ns}base_link"/>
-    <child link="${ns}wheel_1"/>
-    <origin rpy="-1.5707 0 0" xyz="0.1 0.15 0"/>
-    <axis xyz="0 0 1" />
+        <parent link="${ns}base_link"/>
+        <child link="${ns}wheel_1"/>
+        <origin rpy="-1.5707 0 0" xyz="0.0 -0.09 -0.0125"/>
+        <axis xyz="0 0 1" />
     </joint>
     <joint name="${ns}base_to_wheel2" type="continuous">
-    <axis xyz="0 0 1" />
-    <anchor xyz="0 0 0" />
-    <limit effort="100" velocity="100" />
-    <parent link="${ns}base_link"/>
-    <child link="${ns}wheel_2"/>
-    <origin rpy="-1.5707 0 0" xyz="-0.1 0.15 0"/>
-    </joint>
-    <joint name="${ns}base_to_wheel3" type="continuous">
-    <parent link="${ns}base_link"/>
-    <axis xyz="0 0 1" />
-    <child link="${ns}wheel_3"/>
-    <origin rpy="-1.5707 0 0" xyz="0.1 -0.15 0"/>
-    </joint>
-    <joint name="${ns}base_to_wheel4" type="continuous">
-    <parent link="${ns}base_link"/>
-    <axis xyz="0 0 1" />
-    <child link="${ns}wheel_4"/>
-    <origin rpy="-1.5707 0 0" xyz="-0.1 -0.15 0"/>
+        <axis xyz="0 0 1" />
+        <parent link="${ns}base_link"/>
+        <child link="${ns}wheel_2"/>
+        <origin rpy="-1.5707 0 0" xyz="-0.0 0.09 -0.0125"/>
+    </joint>
+    <joint name="${ns}base_to_front_omni" type="fixed">
+        <parent link="${ns}base_link"/>
+        <child link="${ns}front_omni"/>
+        <origin rpy="0 0 0" xyz="0.10 0 -0.05"/>
+    </joint>
+    <joint name="${ns}base_to_back_omni" type="fixed">
+        <parent link="${ns}base_link"/>
+        <child link="${ns}back_omni"/>
+        <origin rpy="0 0 0" xyz="-0.10 0 -0.05"/>
     </joint>
     <joint name="${ns}base_to_laser" type="fixed">
@@ -164,5 +178,5 @@
         <child link="${ns}hokuyo_link"/>
         <axis xyz="0 1 0" />
-        <origin xyz="0.125 0.05 0.135" rpy="0 0 0"/>
+        <origin xyz="0.125 0.0 0.085" rpy="0 0 0"/>
     </joint>
         <gazebo reference="${ns}base_link">
@@ -170,21 +184,45 @@
     </gazebo>
     <gazebo reference="${ns}wheel_1">
-        <material>Gazebo/Gray</material>
+        <material>Gazebo/Grey</material>
     </gazebo>
     <gazebo reference="${ns}wheel_2">
-        <material>Gazebo/Gray</material>
-    </gazebo>
-    <gazebo reference="${ns}wheel_3">
-        <material>Gazebo/Gray</material>
-    </gazebo>
-    <gazebo reference="${ns}wheel_4">
-        <material>Gazebo/Gray</material>
+        <material>Gazebo/Grey</material>
+    </gazebo>
+    <gazebo reference="${ns}front_omni">
+        <material>Gazebo/Grey</material>
+    </gazebo>
+    <gazebo reference="${ns}back_omni">
+        <material>Gazebo/Grey</material>
     </gazebo>
     <gazebo>
         <plugin name="${ns}gazebo_ros_control" filename="libgazebo_ros_control.so">
-        <robotNamespace>${ns}</robotNamespace>
+            <robotNamespace>${ns}</robotNamespace>
+<!--             <robotSimType>gazebo_ros_control/DefaultRobotHWSim</robotSimType>
+            <legacyModeNS>true</legacyModeNS> -->
         </plugin>
     </gazebo>
     <gazebo>
+        <plugin name="differential_drive_controller" filename="libgazebo_ros_diff_drive.so">
+            <alwaysOn>true</alwaysOn>
+            <updateRate>100</updateRate>
+            <leftJoint>${ns}base_to_wheel1</leftJoint>
+            <rightJoint>${ns}base_to_wheel2</rightJoint>
+            <wheelSeparation>0.18</wheelSeparation>
+            <wheelDiameter>${radius_wheel}</wheelDiameter>
+            <commandTopic>cmd_vel</commandTopic>
+            <odometryTopic>odom</odometryTopic>
+            <odometryFrame>odom</odometryFrame>
+            <publishWheelTF>true</publishWheelTF>
+            <publishOdomTF>true</publishOdomTF>
+            <wheelTorque>10</wheelTorque>
+            <legacyMode>true</legacyMode>
+            <publishWheelJointState>true</publishWheelJointState>
+            <wheelAcceleration>2</wheelAcceleration>
+            <robotBaseFrame>base_link</robotBaseFrame>
+            <publishTF>true</publishTF>
+        </plugin>
+    </gazebo>
+    <!--
+     <gazebo>
         <plugin name="${ns}skid_steer_drive_controller" filename="libgazebo_ros_skid_steer_drive.so">
             <updateRate>100.0</updateRate>
@@ -236,3 +274,4 @@
         </sensor>
     </gazebo>
+    -->
 </robot>
